Commit message: 添加底盘接口

File: agv_urdf_test/urdf/agv_urdf_test.urdf (robot description, URDF)
Before this commit: robot agv_urdf_test, 14 links, 13 joints
Joints:
- joint joint_turn_2: limit lower=-6.28 upper=6.28 effort=3 velocity=4 -> (none); type revolute -> continuous
- joint joint_turn_4: limit lower=-6.28 upper=6.28 effort=3 velocity=4 -> (none); type revolute -> continuous

Commit message: 测试了robothw和roscontrol的通断

File: agv_urdf_test/urdf/agv_urdf_test.urdf (robot description, URDF)
Before this commit: robot agv_urdf_test, 14 links, 13 joints
Links:
- link base_link: mass 1008.2 -> 50.2
Joints:
- joint joint_turn_1: limit lower=-6.28 upper=6.28 effort=3 velocity=4 -> effort=3 velocity=4; origin xyz=0.255 0.325 -0.285 rpy=0 0 0 -> xyz=0.255 0.325 -0.285 rpy=0 0 3.1415; type revolute -> continuous
- joint joint_turn_3: limit lower=-6.28 upper=6.28 effort=3 velocity=4 -> effort=3 velocity=4; origin xyz=-0.255 -0.325 -0.285 rpy=0 0 0 -> xyz=-0.255 -0.325 -0.285 rpy=0 0 3.1415; type revolute -> continuous

Commit message: 增加了里程计和imu融合,还有一些bug

File: agv_urdf_test/urdf/agv_urdf_test.urdf (robot description, URDF)
Before this commit: robot agv_urdf_test, 14 links, 13 joints
Links:
- added link link_imu
Joints:
- added joint joint_link_imu: type fixed, parent base_link, child link_imu, origin xyz=0 0 0.03 rpy=0 0 1.5708

Commit message: 更改了amcl全向移动设置

File: agv_urdf_test/urdf/agv_urdf_test.urdf (robot description, URDF)
Before this commit: robot agv_urdf_test, 15 links, 14 joints
Links:
- link base_link: mass 50.2 -> 1.2

Commit message: 加了点东西

File: agv_urdf_test/urdf/agv_urdf_test.urdf (robot description, URDF)
Before this commit: robot agv_urdf_test, 15 links, 14 joints
Joints:
- joint joint_camera: origin xyz=0 0.64 -0.01 rpy=0 0 1.5708 -> xyz=0.5 0 0.01 rpy=0 0 0

Commit message: 运动学换回以前的算法

File: agv_urdf_test/urdf/agv_urdf_test.urdf (robot description, URDF)
Before this commit: robot agv_urdf_test, 15 links, 14 joints
Links:
- removed link link_wheel_2
Joints:
- removed joint joint_wheel_2
