Commit message: 更新了run_all雷达话题,坐标系统一

File: agv_real/urdf/agv_real.urdf (robot description, URDF)
Before this commit: robot agv_real, 15 links, 14 joints
Links:
- removed link link_laser_1
- removed link link_laser_2
- added link laser_1
- added link laser_2
Joints:
- joint joint_laser_1: child link_laser_1 -> laser_1
- joint joint_laser_2: child link_laser_2 -> laser_2

Commit message: 修改真实的雷达参数

File: agv_real/urdf/agv_real.urdf (robot description, URDF)
Before this commit: robot agv_real, 15 links, 14 joints
Joints:
- joint joint_laser_1: origin xyz=0.4 0.5 0.03 rpy=0 0 1.5708 -> xyz=0.586 0.486 0.04 rpy=3.1415 0 2.355
- joint joint_laser_2: origin xyz=-0.4 -0.5 0.03 rpy=0 0 1.5708 -> xyz=-0.586 -0.486 0.04 rpy=3.1415 0 -0.7865

Commit message: 更改了雷达,解决了雷达坐标系和文档中不一致的问题

File: agv_real/urdf/agv_real.urdf (robot description, URDF)
Before this commit: robot agv_real, 15 links, 14 joints
Joints:
- joint joint_laser_1: origin xyz=0.586 0.486 0.04 rpy=3.1415 0 2.355 -> xyz=0.586 0.486 0.04 rpy=3.1415 0 0.7853981
- joint joint_laser_2: origin xyz=-0.586 -0.486 0.04 rpy=3.1415 0 -0.7865 -> xyz=-0.586 -0.486 0.04 rpy=3.1415 0 -2.356194

Commit message: 修改了很多bug

File: agv_real/urdf/agv_real.urdf (robot description, URDF)
Before this commit: robot agv_real, 15 links, 14 joints
Joints:
- joint joint_link_imu: origin xyz=0 0 0.03 rpy=0 0 1.5708 -> xyz=0 0 0.03 rpy=0 0 0

Commit message: Merge #1 into main from dev
fix: detect flag

* dev: (100 commits squashed)

  - 上下回零

  - 上下回零

  - 111

  - 差导航的版本

  - 除了导航的版本

  - 停下bug

  - 把速度滤波曲调

  - 修改了一些小错误

  - fix: delet yolo_ros

  - fix: submodule reload

  - 更改运动学

  - 更改了运动学

  - 更改了正运动学

  - 测试夹爪抬升版本

  - 手动测试夹爪版本

  - 手动测试夹爪版本-1

  - feat: grab lift

  - fix: teb param

  - 放开了限制

  - 1

  - fix: Hfsm stop movebase simple goal

  - feat: ArUco

  - 新的相对运动代码

  - 修改了相对运动

  - 加入获取目标

  - 修改了一些细节

  - 相对运动改好了

  - feat: relative move

  - tiny fix

  - Merge branch &#39;dev&#39; of jihulab.com:xjtu_robot_wx/wangxiao/agv_sim into dev

  - 测试夹爪开合

  - 稳定版本

  - fix: Stop

  - “稳定版本”

  - 测试前转向轮回零

  - fix: hfsm

  - 更新了相对运动视觉的代码

  - 添加了单独编译操作注释

  - 111

  - feat: horizon test

  - Merge branch &#39;dev&#39; of jihulab.com:xjtu_robot_wx/wangxiao/agv_sim into dev

  - fix: Eigen path could not be found

  - 更改了dwa规划

  - 更改真实movebase为测试文件

  - feat: add YoloResult.msg

  - 打开了视觉接口

  - Merge branch &#39;dev&#39; of jihulab.com:xjtu_robot_wx/wangxiao/agv_sim into dev

  - fix: YoloResult.msg

  - 手臂单独运动,但是底盘还会动的bug改掉了

  - Merge branch &#39;dev&#39; of jihulab.com:xjtu_robot_wx/wangxiao/agv_sim into dev

  - 更改了姿态误差计算

  - 更新了注释

  - fix: relative move feedback process

  - Merge branch &#39;dev&#39; of https://jihulab.com/xjtu_robot_wx/wangxiao/agv_sim into dev

  - 添加了点动模式

  - fix reltiv move err define

  - 解决了tfeigen的bug

  - fix: relative move feedback

  - 加了启动文件和tf发布

  - 相对运动的主程序改掉了bug

  - fix: relative move server

  - 更新

  - 添加状态机注释

  - Merge branch &#39;dev&#39; of jihulab.com:xjtu_robot_wx/wangxiao/agv_sim into dev

  - 修改了状态机里面的run函数,并添加了好多函数

  - 修改了main函数入口参数

  - 更改了bug

  - 修改了状态机

  - 优化了状态机,分文件编写

  - fix : visual

  - 000

  - 测试取料

  - 重新标定

  - 正在增加放料代码

  - Merge branch &#39;dev&#39; of jihulab.com:xjtu_robot_wx/wangxiao/agv_sim into dev

  - 修改了状态机

  - 调bug

  - Merge branch &#39;dev&#39; of jihulab.com:xjtu_robot_wx/wangxiao/agv_sim into dev

  - 状态机增加了几个点,顺了一下逻辑

  - 修改了状态机流程

  - 修改了高度和宽度

  - Merge branch &#39;dev&#39; of https://jihulab.com/xjtu_robot_wx/wangxiao/agv_sim into dev

  - feat: add mech-mind camera ros driver

  - fix: new submodule link

  - fix: add submodule command

  - feat: start mech camera

  - fix: hardware respawn automatically

  - fix: hardware launch

  - feat: hfsm add hardware init state

  - feat: PCI error log

  - fix: hfsm add charge&amp;idle

  - fix: camera ip

  - feat: camera service call

  - fix: func name

  - fix: agv_real.launch

  - fix: wheel reset flag

  - fix: shutdown nav&amp;vision roslaunch

  - fix: yolo result reslove

  - fix: detect flag

  - Merge branch main into dev

Signed-off-by: 雪满长安5997284635 <accounts_659e5426a1dd18687695c8bb@mail.teambition.com>
Reviewed-by: 雪满长安5997284635 <accounts_659e5426a1dd18687695c8bb@mail.teambition.com>
Merged-by: 雪满长安5997284635 <accounts_659e5426a1dd18687695c8bb@mail.teambition.com>

CR-link: https://codeup.aliyun.com/657e5b45b488fff322e7d116/xjtu_robot_wx/wangxiao/agv_sim/change/1

File: agv_real/urdf/agv_real.urdf (robot description, URDF)
Before this commit: robot agv_real, 15 links, 14 joints
Links:
- removed link link_camera
- added link camera1_link
Joints:
- joint camera_joint_fake: parent link_camera -> camera1_link
- joint joint_camera: child link_camera -> camera1_link

Commit message: 重新扫描地图

File: agv_real/urdf/agv_real.urdf (robot description, URDF)
Before this commit: robot agv_real, 15 links, 14 joints
Joints:
- joint joint_laser_1: origin xyz=0.586 0.486 0.04 rpy=3.1415 0 0.7853981 -> xyz=0.586 0.486 0.04 rpy=3.1415 0 0.70
